File: PCB/hackpad.kicad_pcb (KiCad board)
At the start: 2 copper layers, 91 x 40.3 mm, 9 parts, among them SW10 RotaryEncoder_Switch_MP, SW4 SW_Push, SW5 SW_Push, SW6 SW_Push, SW7 SW_Push, SW8 SW_Push, SW9 SW_Push, U1 XIAO-RP2040-DIP

Commit message: Changed Rotary Encoder from MP to non-MP
Parts:
- SW0: renamed from SW10; value RotaryEncoder_Switch_MP -> RotaryEncoder_Switch
Connections:
- SW0 pad MP: GND -> (no net)
Routing:
- net GND: track 291.8 -> 237.1 mm
Changed lines of the file:
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@@
 		(descr "Alps rotary encoder, EC11E... with switch, vertical shaft, http://www.alps.com/prod/info/E/HTML/Encoder/Incremental/EC11/EC11E15204A3.html")
 		(tags "rotary encoder")
-		(property "Reference" "SW10"
+		(property "Reference" "SW0"
 			(at 2.8 -4.7 0)
 			(layer "F.SilkS")
@@
 			)
 		)
-		(property "Value" "RotaryEncoder_Switch_MP"
+		(property "Value" "RotaryEncoder_Switch"
 			(at 7.31875 -6.6875 0)
 			(layer "F.Fab")
@@
 			)
 		)
-		(property "Description" "Rotary encoder, dual channel, incremental quadrate outputs, with switch and MP Pin"
+		(property "Description" "Rotary encoder, dual channel, incremental quadrate outputs, with switch"
 			(at 0 0 0)
 			(unlocked yes)
@@
 			(layers "*.Cu" "*.Mask")
 			(remove_unused_layers no)
-			(net 1 "GND")
-			(pinfunction "MP")
-			(pintype "passive")
 		)
 		(pad "MP" thru_hole rect
@@
 			(layers "*.Cu" "*.Mask")
 			(remove_unused_layers no)
-			(net 1 "GND")
-			(pinfunction "MP")
-			(pintype "passive")
 		)
 		(pad "S1" thru_hole circle
@@
 	)
 	(segment
-		(start 106.927876 32.43325)
-		(end 104.81094 32.43325)
-		(width 0.2)
-		(layer "F.Cu")
-		(net 1)
-	)
-	(segment
 		(start 30.50775 48.046564)
 		(end 30.50775 39.492066)
@@
 	)
 	(segment
-		(start 97.88125 39.36294)
-		(end 97.88125 46.7875)
-		(width 0.2)
-		(layer "F.Cu")
-		(net 1)
-	)
-	(segment
 		(start 31.328436 48.86725)
 		(end 30.50775 48.046564)
@@
 	)
 	(segment
+		(start 97.4125 52.3875)
+		(end 90.38125 52.3875)
+		(width 0.2)
+		(layer "F.Cu")
+		(net 1)
+	)
+	(segment
 		(start 38.25875 44.92625)
 		(end 36.430064 44.92625)
@@
 	)
 	(segment
-		(start 104 27.1275)
-		(end 104 38.76875)
-		(width 0.2)
-		(layer "F.Cu")
-		(net 1)
-	)
-	(segment
-		(start 107.60325 48.2655)
-		(end 97.88125 57.9875)
+		(start 105.25125 25.87625)
+		(end 104 27.1275)
 		(width 0.2)
 		(layer "F.Cu")
@@
 	)
 	(segment
-		(start 104 38.76875)
-		(end 90.38125 52.3875)
-		(width 0.2)
-		(layer "F.Cu")
-		(net 1)
-	)
-	(segment
-		(start 105.25125 25.87625)
-		(end 104 27.1275)
+		(start 104 27.1275)
+		(end 104 45.8)
+		(width 0.2)
+		(layer "F.Cu")
+		(net 1)
+	)
+	(segment
+		(start 104 45.8)
+		(end 97.4125 52.3875)
 		(width 0.2)
 		(layer "F.Cu")
@@
 		(width 0.2)
 		(layer "F.Cu")
-		(net 1)
-	)
-	(segment
-		(start 107.60325 27.614624)
-		(end 107.60325 48.2655)
-		(width 0.2)
-		(layer "F.Cu")
-		(net 1)
-	)
-	(segment
-		(start 104.81094 32.43325)
-		(end 97.88125 39.36294)
-		(width 0.2)
-		(layer "F.Cu")
-		(net 1)
-	)
-	(segment
-		(start 110.31775 29.043376)
-		(end 106.927876 32.43325)
-		(width 0.2)
-		(layer "F.Cu")
-		(net 1)
-	)
-	(segment
-		(start 110 29.043376)
-		(end 110.31775 29.043376)
-		(width 0.2)
-		(layer "F.Cu")
